File: tests/fixtures/example_schematic.kicad_sch (KiCad schematic)
At the start: 5 parts, among them J1 Conn_01x04, U1 ESP32-WROOM-32

Commit message: feat: extract component flags (dnp, in_bom, on_board, exclude_from_sim)
Parse KiCad's 4 boolean component flags from .kicad_sch files.
Show DNP/In BOM columns in component listing when non-default values
exist. Add filter_dnp parameter to list_schematic_components.

Also fix tool tests to use .fn for FunctionTool compatibility.
Parts:
- added R3: 0R, Resistor_SMD:R_0402_1005Metric, symbol Device:R
Changed lines of the file:
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@@
     (pin "4")
+  )
+  (symbol (lib_id "Device:R") (at 300 100 0) (unit 1)
+    (exclude_from_sim no) (in_bom no) (on_board yes) (dnp yes)
+    (property "Reference" "R3" (at 295 95 0)
+      (effects (font (size 1.27 1.27)))
+    )
+    (property "Value" "0R" (at 295 105 0)
+      (effects (font (size 1.27 1.27)))
+    )
+    (property "Footprint" "Resistor_SMD:R_0402_1005Metric" (at 300 100 0)
+      (effects (font (size 1.27 1.27)) hide)
+    )
+    (pin "1")
+    (pin "2")
   )
   (net (code 1) (name "GND")
